File: kidcad_folders/NOVAL_PA5-1/NOVAL_PA5-1.kicad_sch (KiCad schematic)
At the start: 10 parts, among them J1 Conn_01x01_Pin, J2 Conn_01x01_Pin, M2 Motor_DC, M3 Motor_DC, M4 Motor_Servo, M5 Motor_DC, M7 Motor_Servo_AirTronics, M8 Motor_Servo_AirTronics, U1 L293D, U2 L293D

Commit message: PA5-1
Parts:
- removed J1, J2: Conn_01x01_Pin, Connector_TE-Connectivity:TE_MATE-N-LOK_1-794374-x_1x01_P4.14mm_Horizontal, symbol Connector:Conn_01x01_Pin
- removed M2, M3, M5: Motor_DC, Connector_PinHeader_2.54mm:PinHeader_1x02_P2.54mm_Vertical, symbol Motor:Motor_DC
- removed M4: Motor_Servo, Connector_PinHeader_2.54mm:PinHeader_1x03_P2.54mm_Vertical, symbol Motor:Motor_Servo
- removed M7, M8: Motor_Servo_AirTronics, Connector_PinHeader_2.54mm:PinHeader_1x03_P2.54mm_Vertical, symbol Motor:Motor_Servo_AirTronics
- added C1, C2, C3, C4: C_US, Capacitor_THT:C_Axial_L5.1mm_D3.1mm_P10.00mm_Horizontal, symbol Device:C_US
- added H1, H2, H3, H4: MountingHole_Pad, MountingHole:MountingHole_2.2mm_M2_DIN965_Pad, symbol Mechanical:MountingHole_Pad
- added HS1: Heatsink, symbol Mechanical:Heatsink
- added J3, J4, J5: Conn_01x03_Pin, Connector_JST:JST_PH_S3B-PH-K_1x03_P2.00mm_Horizontal, symbol Connector:Conn_01x03_Pin
- added J6, J7, J8, J9: Conn_01x02_Pin, Connector_JST:JST_EH_S2B-EH_1x02_P2.50mm_Horizontal, symbol Connector:Conn_01x02_Pin
- added U3, U4: L7805, Package_TO_SOT_THT:TO-220-3_Vertical, symbol Regulator_Linear:L7805
Connections:
- net 11.1V: now also C1.1, C3.1, J9.2 (Pin_2), U3.1 (IN), U4.1 (IN); no longer U1.16 (VCC1), U1.8 (VCC2), U2.16 (VCC1), U2.8 (VCC2)
- net BDIRECTION1: now also J3.3 (Pin_3)
- net BDIRECTION2: now also J4.3 (Pin_3)
- net BDIRECTION3: now also J5.3 (Pin_3)
- net FDIRECTION1: now also J3.2 (Pin_2)
- net FDIRECTION2: now also J4.2 (Pin_2)
- net FDIRECTION3: now also J5.2 (Pin_2)
- net GND: now also C1.2, C2.2, C3.2, C4.2, H1.1, H2.1, H3.1, H4.1, J9.1 (Pin_1), U3.2 (GND), U4.2 (GND)
- net MOTOR1A: now also J6.1 (Pin_1)
- net MOTOR1B: now also J6.2 (Pin_2)
- net MOTOR2A: now also J7.1 (Pin_1)
- net MOTOR2B: now also J7.2 (Pin_2)
- net MOTOR3A: now also J8.1 (Pin_1)
- net MOTOR3B: now also J8.2 (Pin_2)
- net PWM1: now also J3.1 (Pin_1)
- net PWM2: now also J4.1 (Pin_1)
- net PWM3: now also J5.1 (Pin_1)
- new net: C2.1, U1.16 (VCC1), U1.8 (VCC2), U3.3 (OUT)
- new net: C4.1, U2.16 (VCC1), U2.8 (VCC2), U4.3 (OUT)
Other:
- moved on the sheet: U1
